File: Memory/RC2014-TECmemory.sch (KiCad schematic (older format))
At the start: 41 parts, among them J1 RC2014_BUS, J2 Page-out Address, J3 ROM Start/Size, U1 AT28C256, U2 62256, U3 74LS688, U4 74LS74, U5 74LS138, U6 74LS00, U8 74LS86

Commit message: Add files via upload
Parts:
- removed D10, D11, D12, D13, D14, D15, D16, D9: 1N4148, Diode_THT:D_DO-35_SOD27_P7.62mm_Horizontal, symbol Diode:1N4148
- added C7: 100n, Capacitor_THT:C_Disc_D6.0mm_W2.5mm_P5.00mm, symbol Device:C_Small
- added D? (x8): 1N4148, Diode_THT:D_DO-35_SOD27_P7.62mm_Horizontal, symbol Diode:1N4148
- added J4: RAM Size, Connector_PinHeader_2.54mm:PinHeader_2x04_P2.54mm_Vertical, symbol Connector_Generic:Conn_02x04_Odd_Even
- renumbered C8 to C6
Connections:
- net +5V: now also R4.2, R5.1, C7.1; no longer R4.1, R5.2
- net BS0: now also J4.7 (Pin_7)
- net BS1: now also J4.5 (Pin_5)
- net BS2: now also J4.3 (Pin_3)
- net BS3: now also J4.1 (Pin_1)
- net D7: no longer U4.12 (2D)
- net GND: now also C7.2
- net USR1: no longer U4.9 (2Q)
- net at J3.2 (Pin_2): now also D?.1 (K)
- net at J3.4 (Pin_4): now also D?.1 (K)
- net at J3.6 (Pin_6): now also D?.1 (K)
- net at J3.8 (Pin_8): now also D?.1 (K)
- net at U8.2, U8.4: now also R4.1, D?.2 (A), D?.2 (A), D?.2 (A), D?.2 (A); no longer R4.2
- net at U3.19 (P=R), U4.3 (1CLK): no longer U4.11 (2CLK)
- net at U8.5, U8.9: now also R5.2, D?.2 (A), D?.2 (A), D?.2 (A), D?.2 (A); no longer R5.1
- new net: D?.1 (K), J4.2 (Pin_2)
- new net: D?.1 (K), J4.4 (Pin_4)
- new net: D?.1 (K), J4.6 (Pin_6)
- new net: D?.1 (K), J4.8 (Pin_8)
- new net INT: U4.9 (2Q)
- new net M1: U4.12 (2D)
Other:
- note added: "In this memory model, the ROM is placed in the upper\nend of the 64k addressable range, while the lower 32K \nis always reserved for RAM.\n\nJ3 lets the user control what size (in 8k blocks) the ROM is\nand at what address range it is to start at.\n\nFor example, if the user has a 16k ROM, that they wish to start\nat the 40K mark, jumpers would be placed on BS5 and BS6."
- note added: "RAM Select"
- note added: "ROM Select"
- note added: "The ROM is selected (asserted LOW)\nIF {\n 1) The Shadow Latch is Low (on reset)\nAND\n 2) Any address in the lower 2K is requested }\nOR\n 3) If an address is within the range determined by J3\nOTHERWISE\n The RAM bank on this card is selected if it falls within the\n address range determined by J4, but must start at $0000"
- note added: "This line is asserted HIGH when the Memory Latch is Low, \nAND all the upper address lines are Low, \nmeaning the CPU is addressing the lowest 2K range,\nwhich is where the TEC-1 ROMs were placed."
- note added: "USR1 is a latched output \nthat can be used for BitBang serial\nor single stepping code."
- note removed: "USR1 is a latched output\nthat can be used for BitBang serial."
- moved on the sheet: U6A, U6B, U8A, U8B, U8C

Commit message: Add files via upload
Parts:
- removed U1: AT28C256, Socket:DIP_Socket-28_W11.9_W12.7_W15.24_W17.78_W18.5_3M_228-1277-00-0602J, symbol ZEC-1:AT28C256
- removed U?: 27C64, Package_DIP:DIP-28_W15.24mm, symbol ZEC-1:27C64
- removed U?: FM16W08-SG, Package_SO:SOIC-28W_7.5x17.9mm_P1.27mm, symbol Memory_NVRAM:FM16W08-SG
- added D?: 1N4148, Diode_THT:D_DO-35_SOD27_P7.62mm_Horizontal, symbol Diode:1N4148
- added R6: 10K, Resistor_THT:R_Axial_DIN0207_L6.3mm_D2.5mm_P10.16mm_Horizontal, symbol Device:R_Small_US
- added SW1: STEP, symbol Switch:SW_SPST
- added U1: AT28C64, Socket:DIP_Socket-28_W11.9_W12.7_W15.24_W17.78_W18.5_3M_228-1277-00-0602J, symbol ZEC-1:AT28C64
Connections:
- net +5V: now also U1.27 (~WE), U1.28 (VCC)
- net A0: now also U1.10 (A0)
- net A1: now also U1.9 (A1)
- net A10: now also U1.21 (A10)
- net A11: now also U1.23 (A11)
- net A12: now also U1.2 (A12)
- net A13: now also U1.26 (NC)
- net A14: now also U1.1 (NC)
- net A2: now also U1.8 (A2)
- net A3: now also U1.7 (A3)
- net A4: now also U1.6 (A4)
- net A5: now also U1.5 (A5)
- net A6: now also U1.4 (A6)
- net A7: now also U1.3 (A7)
- net A8: now also U1.25 (A8)
- net A9: now also U1.24 (A9)
- net D0: now also U1.11 (D0)
- net D1: now also U1.12 (D1)
- net D2: now also U1.13 (D2)
- net D3: now also U1.15 (D3)
- net D4: now also U1.16 (D4)
- net D5: now also U1.17 (D5)
- net D6: now also U1.18 (D6)
- net D7: now also U1.19 (D7)
- net GND: now also R6.1, U1.14 (GND)
- net M1: now also U4.11 (2CLK); no longer U4.12 (2D)
- net RD: now also U1.22 (~OE)
- net at U6.6: now also D?.2 (A), U1.20 (~CS)
- new net: R6.2, SW1.1 (A), U4.12 (2D)
- new net: D?.1 (K), SW1.2 (B)
Other:
- note added: "This FlipFlop used for Single Stepping\nthrough Code, triggering INT on each memory\nread cycle if the ROM is not selected.\nUse the switch to disable Stepper."
- note added: "To remove the Shadowed ROM, an OUTput of $00\nto the Port specified by the jumpers Flips the\nFlop off and removes the ROM from lower 2K.\n(It is possible to Shadow it back in with an OUTput of $01)"
- note added: "on = ROM Shadowed"
- note removed: "USR1 is a latched output \nthat can be used for BitBang serial\nor single stepping code."
Changed lines of the file:
@@
 encoding utf-8
 Sheet 1 1
-Title ""
-Date ""
-Rev ""
-Comp ""
+Title "TEC-2014 Memory"
+Date "2021-07-20"
+Rev "v.1.0"
+Comp "Mark Jelic, 2021"
 Comment1 ""
 Comment2 ""
-Comment3 ""
-Comment4 ""
+Comment3 "by John Hardy & Ken Stone, 1983"
+Comment4 "Based on the design of the TEC-1"
 $EndDescr
 $Comp
@@
 Wire Wire Line
 	11975 4800 8425 4800
-Wire Wire Line
-	7400 5275 7400 5125
-Text GLabel 7400 5125 2    50   Input ~ 0
+Text GLabel 7400 5275 1    50   Input ~ 0
 +5V
-Wire Wire Line
-	6900 6025 6875 6025
-Wire Wire Line
-	6875 6025 6875 5525
-Wire Wire Line
-	6875 5525 6900 5525
-Wire Wire Line
-	6875 5525 6875 5125
-Wire Wire Line
-	6875 5125 7400 5125
-Connection ~ 6875 5525
 $Comp
 L ZEC-1:74LS688 U3
@@
 Wire Wire Line
 	8625 2450 8400 2450
-Wire Wire Line
-	5750 5350 4700 5350
-Entry Wire Line
-	6650 5725 6550 5625
-Text Label 6650 5725 0    50   ~ 0
+Entry Wire Line
+	6650 6225 6550 6125
+Text Label 6650 5625 0    50   ~ 0
 M1
 Wire Wire Line
-	6900 5725 6650 5725
-Entry Wire Line
-	6550 6125 6650 6225
+	6900 6225 6650 6225
 Text Label 6650 6225 0    50   ~ 0
 D0
-Wire Wire Line
-	6900 6225 6650 6225
 Entry Wire Line
 	6550 7700 6650 7800
@@
 Text Label 6650 5425 0    50   ~ 0
 RESET
-Wire Wire Line
-	6900 6125 6725 6125
-Wire Wire Line
-	6725 6125 6725 6025
-Wire Wire Line
-	6725 6025 5750 6025
 Wire Wire Line
 	6900 5625 6650 5625
@@
 Wire Wire Line
 	8225 8100 8525 8100
-Text Notes 7800 6025 0    50   ~ 0
+Text Notes 7950 6025 0    50   ~ 0
 On RESET, Q=Lo
 $Comp
 L power:GND #PWR0115
 U 1 1 5FB8FA4F
-P 8725 6225
-F 0 "#PWR0115" H 8725 5975 50  0001 C CNN
-F 1 "GND" H 8730 6052 50  0000 C CNN
-F 2 "" H 8725 6225 50  0001 C CNN
-F 3 "" H 8725 6225 50  0001 C CNN
-	1    8725 6225
+P 8850 5975
+F 0 "#PWR0115" H 8850 5725 50  0001 C CNN
+F 1 "GND" H 8855 5802 50  0000 C CNN
+F 2 "" H 8850 5975 50  0001 C CNN
+F 3 "" H 8850 5975 50  0001 C CNN
+	1    8850 5975
 	-1   0    0    -1
 $EndComp
-Wire Wire Line
-	7850 5925 7925 5925
 $Comp
 L Diode:1N4148 D3
 U 1 1 5FC81AE3
-P 8225 6600
-F 0 "D3" H 8225 6816 50  0001 C CNN
-F 1 "1N4148" H 8225 6725 50  0001 C CNN
-F 2 "Diode_THT:D_DO-35_SOD27_P7.62mm_Horizontal" H 8225 6425 50  0001 C CNN
-F 3 "https://assets.nexperia.com/documents/data-sheet/1N4148_1N4448.pdf" H 8225 6600 50  0001 C CNN
-	1    8225 6600
+P 8075 6600
+F 0 "D3" H 8075 6816 50  0001 C CNN
+F 1 "1N4148" H 8075 6725 50  0001 C CNN
+F 2 "Diode_THT:D_DO-35_SOD27_P7.62mm_Horizontal" H 8075 6425 50  0001 C CNN
+F 3 "https://assets.nexperia.com/documents/data-sheet/1N4148_1N4448.pdf" H 8075 6600 50  0001 C CNN
+	1    8075 6600
 	-1   0    0    1
 $EndComp
@@
 	8775 7100 8375 7100
 Wire Wire Line
-	8075 6600 7925 6600
-Wire Wire Line
-	7925 5925 7925 6600
-Wire Wire Line
 	6650 6800 8075 6800
 Wire Wire Line
@@
 Text Label 8225 8400 0    50   ~ 0
 BS2
-$Comp
-L ZEC-1:AT28C256 U1
-U 1 1 6008D3E3
-P 7400 3350
-F 0 "U1" H 7650 4400 50  0000 C CNN
-F 1 "AT28C256" V 7400 3350 50  0000 C CNB
-F 2 "Socket:DIP_Socket-28_W11.9_W12.7_W15.24_W17.78_W18.5_3M_228-1277-00-0602J" H 7400 3350 50  0001 C CNN
-F 3 "http://ww1.microchip.com/downloads/en/DeviceDoc/doc0006.pdf" H 7400 3350 50  0001 C CNN
-	1    7400 3350
-	1    0    0    -1
-$EndComp
 Wire Wire Line
 	6775 4250 6900 4250
@@
 	6650 5925 6900 5925
 Entry Wire Line
-	6550 4875 6650 4975
-Text Label 6650 4975 0    50   ~ 0
+	6550 4900 6650 5000
+Text Label 6650 5000 0    50   ~ 0
 INT
-Wire Wire Line
-	7850 5475 7850 4975
-Wire Wire Line
-	6650 4975 7850 4975
 $Comp
 L Device:R_Small_US R1
@@
 Wire Wire Line
 	8625 5725 8725 5725
-$Comp
-L power:GND #PWR0101
-U 1 1 5FEAE0F7
-P 8725 5725
-F 0 "#PWR0101" H 8725 5475 50  0001 C CNN
-F 1 "GND" H 8730 5552 50  0000 C CNN
-F 2 "" H 8725 5725 50  0001 C CNN
-F 3 "" H 8725 5725 50  0001 C CNN
-	1    8725 5725
-	-1   0    0    -1
-$EndComp
 Entry Wire Line
 	1700 5875 1800 5975
@@
 	0    -1   -1   0
 $EndComp
-Text Notes 7875 5250 0    50   ~ 0
-USR1 is a latched output \nthat can be used for BitBang serial\nor single stepping code.
-$Comp
-L ZEC-1:27C64 U?
-U 1 1 60485EF0
-P 11025 3225
-F 0 "U?" H 11025 4406 50  0000 C CNN
-F 1 "27C64" H 11025 4315 50  0000 C CNB
-F 2 "Package_DIP:DIP-28_W15.24mm" V 11075 3150 50  0001 C CNN
-F 3 "http://ww1.microchip.com/downloads/en/DeviceDoc/11107M.pdf" H 11025 3225 50  0001 C CNN
-	1    11025 3225
-	1    0    0    -1
-$EndComp
-$Comp
-L Memory_NVRAM:FM16W08-SG U?
-U 1 1 604882A5
-P 12525 2950
-F 0 "U?" H 12525 3931 50  0000 C CNN
-F 1 "FM16W08-SG" H 12525 3840 50  0000 C CNN
-F 2 "Package_SO:SOIC-28W_7.5x17.9mm_P1.27mm" H 12525 2950 50  0001 C CNN
-F 3 "http://www.cypress.com/file/41731/download" H 12525 2950 50  0001 C CNN
-	1    12525 2950
-	1    0    0    -1
-$EndComp
+Text Notes 7875 5350 0    50   ~ 0
+This FlipFlop used for Single Stepping\nthrough Code, triggering INT on each memory\nread cycle if the ROM is not selected.\nUse the switch to disable Stepper.
 Text Notes 9300 6900 0    50   ~ 0
 This line is asserted HIGH when the Memory Latch is Low, \nAND all the upper address lines are Low, \nmeaning the CPU is addressing the lowest 2K range,\nwhich is where the TEC-1 ROMs were placed.
@@
 Wire Wire Line
 	3625 6800 3725 6800
-Wire Wire Line
-	5750 5350 5750 6025
-Entry Wire Line
-	6650 5625 6550 5525
+Text GLabel 6900 5525 0    50   Input ~ 0
++5V
+Entry Wire Line
+	6550 5525 6650 5625
+Wire Wire Line
+	7850 5000 7850 5475
+Wire Wire Line
+	7850 5925 7925 5925
+Wire Wire Line
+	7925 5925 7925 6600
+Wire Wire Line
+	6775 4700 6350 4700
+Connection ~ 6775 4700
+Wire Wire Line
+	8725 5725 8725 5975
+Wire Wire Line
+	8850 5975 8725 5975
+Connection ~ 8725 5975
+Wire Wire Line
+	8725 5975 8725 6225
+Text GLabel 6900 6025 0    50   Input ~ 0
++5V
+Wire Wire Line
+	8375 6600 8225 6600
+Wire Wire Line
+	7850 5000 6650 5000
+Wire Wire Line
+	4700 6050 6625 6050
+Wire Wire Line
+	6625 6050 6625 6125
+Wire Wire Line
+	6625 6125 6900 6125
+Wire Wire Line
+	6350 5725 6900 5725
+$Comp
+L Device:R_Small_US R6
+U 1 1 61A44B98
+P 6250 5725
+F 0 "R6" V 6150 5725 50  0000 C CNN
+F 1 "10K" V 6350 5725 50  0000 C CNN
+F 2 "Resistor_THT:R_Axial_DIN0207_L6.3mm_D2.5mm_P10.16mm_Horizontal" H 6250 5725 50  0001 C CNN
+F 3 "~" H 6250 5725 50  0001 C CNN
+	1    6250 5725
+	0    -1   -1   0
+$EndComp
+$Comp
+L Switch:SW_SPST SW1
+U 1 1 61ABE92E
+P 6350 5275
+F 0 "SW1" H 6350 5225 50  0000 C CNN
+F 1 "STEP" H 6350 5419 50  0000 C CNN
+F 2 "" H 6350 5275 50  0001 C CNN
+F 3 "~" H 6350 5275 50  0001 C CNN
+	1    6350 5275
+	0    -1   -1   0
+$EndComp
+Wire Wire Line
+	4700 5350 4700 6050
+$Comp
+L power:GND #PWR?
+U 1 1 61BE6569
+P 6150 5725
+F 0 "#PWR?" H 6150 5475 50  0001 C CNN
+F 1 "GND" H 6155 5552 50  0000 C CNN
+F 2 "" H 6150 5725 50  0001 C CNN
+F 3 "" H 6150 5725 50  0001 C CNN
+	1    6150 5725
+	-1   0    0    -1
+$EndComp
+Wire Wire Line
+	6350 5475 6350 5725
+Connection ~ 6350 5725
+$Comp
+L Diode:1N4148 D?
+U 1 1 61C2E977
+P 6350 4850
+F 0 "D?" H 6350 5066 50  0001 C CNN
+F 1 "1N4148" H 6350 4975 50  0001 C CNN
+F 2 "Diode_THT:D_DO-35_SOD27_P7.62mm_Horizontal" H 6350 4675 50  0001 C CNN
+F 3 "https://assets.nexperia.com/documents/data-sheet/1N4148_1N4448.pdf" H 6350 4850 50  0001 C CNN
+	1    6350 4850
+	0    -1   -1   0
+$EndComp
+Wire Wire Line
+	6350 5075 6350 5000
+Text Notes 8550 6350 0    50   ~ 0
+on = ROM Shadowed
+Text Notes 3950 3900 0    50   ~ 0
+To remove the Shadowed ROM, an OUTput of $00\nto the Port specified by the jumpers Flips the\nFlop off and removes the ROM from lower 2K.\n(It is possible to Shadow it back in with an OUTput of $01)
+$Comp
+L ZEC-1:AT28C64 U1
+U 1 1 61DD86E5
+P 7400 3350
+F 0 "U1" H 7650 4400 50  0000 C CNN
+F 1 "AT28C64" V 7400 3350 50  0000 C CNB
+F 2 "Socket:DIP_Socket-28_W11.9_W12.7_W15.24_W17.78_W18.5_3M_228-1277-00-0602J" H 7400 3350 50  0001 C CNN
+F 3 "http://ww1.microchip.com/downloads/en/DeviceDoc/doc0006.pdf" H 7400 3350 50  0001 C CNN
+	1    7400 3350
+	1    0    0    -1
+$EndComp
 Wire Bus Line
 	9975 1875 9975 3050
